File: boards/daughterboard/pcie_board.sch (EAGLE design)
At the start: 61 parts, among them IC1 XMEGA16A4A, IC2 SN754410, T1 2N3704, T2 2N3704, T3 2N3704, T4 2N3704, T5 2N3704, T6 2N3704, T7 2N3704, X1 PCI-E1X_EDGE

Commit message: Latest board(the one presented at class
Parts:
- removed ANALOG_IN, JTAG: (no value), pinhead:PINHD-2X3
- removed ASYNC_INT_IN: (no value), pinhead:PINHD-2X2
- removed C1, C2: (no value), capacitor-wima:C2.5/4
- removed LED_ERROR, LED_MOT_A, LED_MOT_B, LED_SELECTED: (no value), led:LED5MM
- removed MOT_A_OUT, MOT_B_OUT, TRIAC_OUT, ZEROCROSS_SENSE: (no value), pinhead:PINHD-1X2
- removed PWR, PWR1, PWR2: (no value), pinhead:PINHD-1X4
- removed S1: (no value), switch-dil:DA05
- removed T1, T2, T3, T4, T5, T6, T7: 2N3704, transistor:2N3704
- added CHANNEL_1_ADC, CHANNEL_2_ADC, I2C1, I2C2, JP4, JP5, JP6, OPTO_IN: (no value), pinhead:PINHD-1X2
- added JP1, JP3: (no value), pinhead:PINHD-2X3
- added JP10, JP11, JP12, JP13, MOTOR_1_OUT, MOTOR_2_OUT: (no value), SparkFun:M023.5MM
- added JP2, JP7, JP8, JP9, SLAVE_SELECT_2: (no value), pinhead:PINHD-1X1
- added LED1, LED2, LED3: (no value), led:LEDCHIP-LED0603
- added LED_ERROR1, LED_ERROR2, LED_MOT1, LED_MOT2: (no value), led:LED5MM
- added MPC3002ADC: (no value), ic-package:DIL8
- added OK3: TIL193, optocoupler:TIL193
- added R29, R30, R31, R32: (no value), resistor:R-US_M0805
- added SPI_OUT: (no value), pinhead:PINHD-1X5
- added U$1: PCI-E1X_EDGE, con-pci_express(pci-e):PCI-E1X_EDGE
- EXTERNAL_POWER_IN: device pinhead:PINHD-1X2 -> SparkFun:M023.5MM
- OK1, OK2: value ILQ620 -> TIL193; device optocoupler:ILQ620 -> optocoupler:TIL193
- R1, R2, R22, R3, R5, R6, R7: value 10K -> (none); device resistor:R-US_R0805 -> resistor:R-US_M0805
- R10, R11, R15, R16, R17, R8, R9: value 47Ohm -> (none); device resistor:R-US_0207/10 -> resistor:R-US_M0805
- R12, R4: value 100Ohm -> (none); device resistor:R-US_0207/10 -> resistor:R-US_M0805
- R13, R14, R18, R19, R20: value 100Ohm -> (none); device resistor:R-US_R0805 -> resistor:R-US_M0805
- R21: value 10K -> (none); device resistor:R-US_0207/10 -> resistor:R-US_M0805
- R23, R24, R25, R26, R27, R28: value 47Ohm -> (none); device resistor:R-US_0204/7 -> resistor:R-US_M0805
- X1: value PCI-E1X_EDGE -> 9090-4R; device con-pci_express(pci-e):PCI-E1X_EDGE -> con-thomas-betts:9090-4R
Connections:
- removed net +12V: PWR.1, PWR1.1, PWR2.1, X1.A3, X1.B3
- removed net +5V: PWR.2, PWR1.2, PWR2.2, X1.A2, X1.B2
- removed net EXT_5V: IC2.VCC1, R1.2, R2.1, R22.2, R3.1, R5.2, R6.1, R7.1, VREG.OUT
- removed net N$15: IC1.PC3, R27.1
- removed net N$4: LED_POWER.A, R23.2
- removed net N$43: IC2.M2A, MOT_B_OUT.1
- removed net N$45: IC1.PC6, S1.7
- removed net N$46: IC1.PC5, S1.6
- removed net N$47: OK2B.AC1, R10.1
- removed net N$48: OK2C.AC1, R11.1
- removed net N$49: OK2B.AC2, T2.C
- removed net N$50: OK2C.AC2, T3.C
- removed net N$51: R12.1, T1.B
- removed net N$52: R13.1, T2.B
- removed net N$53: R14.1, T3.B
- removed net N$55: IC1.PD3, R14.2
- removed net N$56: IC1.PD4, R13.2
- removed net N$57: OK1A.AC2, T4.C
- removed net N$58: OK1B.AC2, T5.C
- removed net N$59: OK1C.AC2, T6.C
- removed net N$60: R18.1, T4.B
- removed net N$61: R19.1, T5.B
- removed net N$62: R20.1, T6.B
- removed net N$65: IC1.PD5, R19.2
- removed net N$66: IC1.PD6, R20.2
- removed net N$67: OK1A.AC1, R15.1
- removed net N$68: OK1B.AC1, R16.1
- removed net N$69: OK1C.AC1, R17.1
- removed net N$70: IC1.PA4, S1.8
- removed net N$71: ANALOG_IN.2, IC1.PB0
- removed net N$73: ANALOG_IN.5, IC1.PA0
- removed net N$74: ANALOG_IN.3, IC1.PA1
- removed net N$75: ASYNC_INT_IN.1, IC1.PA2
- removed net N$77: IC1.PA5, R23.1
- removed net PWM_A: IC1.PD1, R12.2
- removed net TRIAC_OUT: IC1.PC7, R4.2
- removed net ZEROCROSS_IN: IC1.PD7, OK2D.C, R21.1
- new net ADC_CLK: MPC3002ADC.7, OK3A.COL, R30.1, SPI_OUT.3
- new net ADC_CS: MPC3002ADC.1, OK1D.COL, R27.1
- new net ADC_MISO: MPC3002ADC.6, R28.1, SPI_OUT.2
- new net ADC_MOSI: MPC3002ADC.5, OK3B.COL, R29.1, SPI_OUT.1
- new net ADC_VSS: CHANNEL_2_ADC.1, IC2.VCC1, LED3.A, R19.2, R20.2, R21.1, R22.2, R23.2, R24.2, R27.2, R29.2, R30.2, R31.2, SPI_OUT.5, VREG.OUT
- new net ANALOG_1: IC1.PA0, JP1.1
- new net ANALOG_2: IC1.PA1, JP1.2
- new net ANALOG_3: IC1.PA3, JP1.3
- new net ANALOG_4: IC1.PA4, JP1.4
- new net ANALOG_5: IC1.PA5, JP1.5
- new net ANALOG_6: IC1.PA6, JP1.6
- new net ASYNC_1: IC1.PD2, JP8.1
- new net ASYNC_2: IC1.PC2, JP2.1
- new net ASYNC_3: IC1.PB2, JP9.1
- new net ASYNC_4: IC1.PA2, JP7.1
- new net CHANNEL_1: CHANNEL_1_ADC.1, MPC3002ADC.2
- new net LED_ERROR1: IC1.PD5, R15.2
- new net LED_ERROR2: IC1.PD6, R16.2
- new net LED_MOT_1: IC1.PD7, R17.2
- new net LED_MOT_2: IC1.PE3, R18.2
- new net LED_ORDERS: IC1.PD4, R14.2
- new net LED_POWER: IC1.PD3, R13.2
- new net MISO: IC1.PC6, OK3C.COL, R4.1
- new net MOSI: IC1.PC5, OK3B.A
- new net MOT_CONTROL_A_1: IC1.PC3, OK1B.A
- new net MOT_CONTROL_A_2: IC1.PB3, OK2B.A
- new net MOT_CONTROL_B_1: IC1.PC4, OK1C.A
- new net MOT_CONTROL_B_2: IC1.PB1, OK2C.A
- new net MOT_CONTROL_EN_1: IC1.PD1, OK1A.A
- new net MOT_CONTROL_EN_2: IC1.PD0, OK2A.A
- new net N$38: JP10.1, JP11.1, X1.1
- new net OPTIONAL_OPTO_IN: OK3D.COL, R8.1
- new net PDI_CLK: IC1.!RESET!/PDI_CLK, JP3.2
- new net PDI_DATA: IC1.PDI_DATA, JP3.6
- new net SCK: IC1.PC7, OK3A.A
- new net SS1: IC1.PA7, OK2D.A
- new net SS2: IC1.PB0, OK1D.A
- net +3V3: now also JP3.5, JP4.1, JP5.1, JP6.1, R4.2, U$1.A1, U$1.A2, U$1.B1, U$1.B2; no longer C1.1, C2.2, JTAG.2, PWR.3, PWR1.3, PWR2.3, R10.2, R11.2, R15.2, R16.2, R17.2, R21.2, R9.2, S1.1, S1.2, S1.3, S1.4, S1.5, X1.A1, X1.B1
- net ERROR: now also IC1.PE2, U$1.A7, U$1.B7; no longer IC1.PD2, X1.A6
- net EXT_MOTOR_GND: now also CHANNEL_2_ADC.2, MPC3002ADC.4, MPC3002ADC.8, OK1A.EMIT, OK1B.EMIT, OK1C.EMIT, OK1D.EMIT, OK2A.EMIT, OK2B.EMIT, OK2C.EMIT, OK2D.EMIT, OK3A.EMIT, OK3B.EMIT, OK3C.C, R25.2, R26.2, R32.2, SPI_OUT.4; no longer OK1A.E, OK1B.E, OK1C.E, OK1D.E, OK2A.E, OK2B.E, OK2C.E, TRIAC_OUT.2
- net GND: now also JP10.2, JP11.2, JP12.2, JP13.2, JP3.1, JP4.2, JP5.2, LED_ERROR1.C, LED_ERROR2.C, LED_MOT1.C, LED_MOT2.C, OK3C.EMIT, OK3D.EMIT, R1.1, R10.1, R11.1, R12.1, R2.1, R3.1, R5.1, R6.1, R7.1, R9.1, U$1.A10, U$1.A11, U$1.A12, U$1.A13, U$1.A14, U$1.A15, U$1.A16, U$1.A17, U$1.A18, U$1.A8, U$1.A9, U$1.B10, U$1.B11, U$1.B12, U$1.B13, U$1.B14, U$1.B15, U$1.B16, U$1.B17, U$1.B18, U$1.B8, U$1.B9, X1.2, X1.3; no longer C1.2, C2.1, JTAG.6, LED_ERROR.C, LED_MOT_A.C, LED_MOT_B.C, LED_SELECTED.C, OK2D.E, PWR.4, PWR1.4, PWR2.4, T1.E, T2.E, T3.E, T4.E, T5.E, T6.E, T7.E, X1.A10, X1.A12, X1.A13, X1.A14, X1.A15, X1.A16, X1.A17, X1.A18, X1.A4, X1.A5, X1.A7, X1.A8, X1.B10, X1.B11, X1.B12, X1.B13, X1.B14, X1.B15, X1.B16, X1.B17, X1.B18, X1.B4, X1.B5, X1.B7, X1.B9
- net N$1: now also IC2.M2A, MOTOR_2_OUT.1; no longer IC1.PA7, R25.1
- net N$10: now also OK2B.C, R6.2; no longer IC1.PE3, R26.1
- net N$11: now also OK2C.C, R7.2; no longer LED_ERROR.A, R26.2
- net N$12: now also OK2D.C, R10.2; no longer ANALOG_IN.4, IC1.PB1
- net N$13: now also OK3A.C, R11.2; no longer ANALOG_IN.6, IC1.PB3
- net N$14: now also OK3B.C, R12.2; no longer ASYNC_INT_IN.3, IC1.PC2
- net N$16: now also LED_POWER.A, R13.1; no longer ANALOG_IN.1, IC1.PA3
- net N$17: now also LED_ORDERS.A, R14.1; no longer IC1.PC4, R28.1
- net N$18: now also CHANNEL_1_ADC.2, MPC3002ADC.3; no longer ASYNC_INT_IN.4, IC1.PE2
- net N$19: now also OK2D.COL, R31.1, SLAVE_SELECT_2.1; no longer LED_MOT_B.A, R28.2
- net N$2: now also JP12.1, JP13.1, X1.4; no longer IC1.!RESET!/PDI_CLK, JTAG.5
- net N$20: now also LED_ERROR1.A, R15.1; no longer IC1.PA6, R24.1
- net N$21: now also LED_ERROR2.A, R16.1; no longer ASYNC_INT_IN.2, IC1.PB2
- net N$22: now also LED_MOT1.A, R17.1; no longer LED_MOT_A.A, R27.2
- net N$23: now also LED_MOT2.A, R18.1; no longer IC1.PR0(XT2), S1.9
- net N$24: now also IC2.EN1, LED2.A, OK1A.COL, R21.2; no longer IC1.PR1(XT1), S1.10
- net N$25: now also IC2.SIG1A, OK1B.COL, R19.1; no longer OK1D.AC2, T7.C
- net N$26: now also LED2.C, R25.1; no longer JTAG.3
- net N$27: now also LED1.C, R26.1; no longer JTAG.4
- net N$28: now also IC2.EN2, LED1.A, OK2A.COL, R20.1; no longer OK2D.AC1, ZEROCROSS_SENSE.1
- net N$29: now also IC2.SIG1B, OK1C.COL, R22.1; no longer OK2A.AC2, T1.C
- net N$3: now also IC2.M2B, MOTOR_2_OUT.2; no longer R4.1, T7.B
- net N$30: now also IC2.SIG2A, OK2B.COL, R24.1; no longer OK2A.AC1, R9.1
- net N$31: now also MOTOR_1_OUT.2; no longer MOT_A_OUT.2
- net N$32: now also MOTOR_1_OUT.1; no longer MOT_A_OUT.1
- net N$33: now also IC2.SIG2B, OK2C.COL, R23.1; no longer IC2.EN1, OK1A.C, R1.1
- net N$34: now also OK3C.A, R28.2; no longer IC2.SIG1A, OK1B.C, R2.2
- net N$35: now also OK3D.A, OPTO_IN.1; no longer IC2.SIG1B, OK1C.C, R3.2
- net N$36: now also OK3D.C, OPTO_IN.2; no longer OK2D.AC2, ZEROCROSS_SENSE.2
- net N$37: now also LED3.C, R32.1; no longer IC1.PD0, R18.2
- net N$39: now also JP3.4; no longer IC2.M2B, MOT_B_OUT.2
- net N$40: now also JP3.3; no longer IC2.EN2, OK2A.C, R5.1
- net N$41: now also IC1.PR0(XT2); no longer IC2.SIG2A, OK2B.C, R6.2
- net N$42: now also IC1.PR1(XT1), JP6.2; no longer IC2.SIG2B, OK2C.C, R7.2
- net N$5: now also OK1A.C, R2.2; no longer OK1D.C, R22.1, TRIAC_OUT.1
- net N$6: now also OK1B.C, R1.2; no longer LED_ORDERS.A, R24.2
- net N$7: now also OK1C.C, R3.2; no longer LED_SELECTED.A, R25.2
- net N$8: now also OK1D.C, R9.2; no longer OK1D.AC1, R8.1
- net N$9: now also OK2A.C, R5.2; no longer IC1.PDI_DATA, JTAG.1
- net SCL1: now also I2C1.1, U$1.A3, U$1.B3; no longer X1.B6
- net SCL2: now also I2C2.1, U$1.A5, U$1.B5; no longer X1.A9
- net SDA1: now also I2C1.2, U$1.A4, U$1.B4; no longer X1.B8
- net SDA2: now also I2C2.2, U$1.A6, U$1.B6; no longer X1.A11
Other:
- moved on the sheet: EXTERNAL_POWER_IN, IC1, LED_ORDERS, LED_POWER, R1, R10, R11, R12, R13, R14, R15, R16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

Commit message: added some fets to take care of the overloaded atxmega.
Parts:
- removed JP10, JP11, JP12, JP13: (no value), SparkFun:M023.5MM
- removed MPC3002ADC: (no value), ic-package:DIL8
- removed VREG: (no value), v-reg:78MXXL
- removed X1: 9090-4R, con-thomas-betts:9090-4R
- added C1, C2: (no value), resistor:C-US025-040X050
- added CHANNEL_3_ADC, CHANNEL_4_ADC: (no value), pinhead:PINHD-1X2
- added IC3: UA78M05DCY, linear:UA78M05DCY
- added OK4, OK5, OK6: LTV826, optocoupler:LTV826
- added Q1, Q2, Q3, Q4, Q5, Q6: FDN360P, transistor-power:FDN360P
- added R33, R34, R35, R36, R37, R38: (no value), resistor:R-US_M0805
- added SENSOR_GND: (no value), SparkFun:M023.5MM
- added U$2: MCP3004, microchip:MCP3004
- OK1, OK2, OK3: value TIL193 -> LTV826; device optocoupler:TIL193 -> optocoupler:LTV826
Connections:
- removed net ADC_VSS: CHANNEL_2_ADC.1, IC2.VCC1, LED3.A, R19.2, R20.2, R21.1, R22.2, R23.2, R24.2, R27.2, R29.2, R30.2, R31.2, SPI_OUT.5, VREG.OUT
- removed net CHANNEL_1: CHANNEL_1_ADC.1, MPC3002ADC.2
- new net CH1: CHANNEL_1_ADC.1, U$2.CH0
- new net CH2: CHANNEL_2_ADC.1, U$2.CH1
- new net CH3: CHANNEL_3_ADC.1, U$2.CH2
- new net CH4: CHANNEL_4_ADC.1, U$2.CH3
- new net EXT_MOTOR_VCC: C1.1, IC2.VCC1, IC3.VO, LED3.A, R19.2, R20.2, R21.1, R22.2, R23.2, R24.2, R27.2, R29.2, R30.2, R31.2, SPI_OUT.5, U$2.VDD, U$2.VREF
- new net N$15: Q3.S, R35.2
- new net N$4: OK1A.C, Q1.D
- net +3V3: now also C2.2, OK1A.A, OK1B.A, OK2A.A, OK2B.A, OK3A.A, OK3B.A
- net ADC_CLK: now also OK5A.COL, SPI_OUT.1, U$2.CLK; no longer MPC3002ADC.7, OK3A.COL, SPI_OUT.3
- net ADC_CS: now also OK4A.COL, U$2.CS; no longer MPC3002ADC.1, OK1D.COL
- net ADC_MISO: now also SPI_OUT.3, U$2.DOUT; no longer MPC3002ADC.6, SPI_OUT.2
- net ADC_MOSI: now also OK5B.COL, SPI_OUT.2, U$2.DIN; no longer MPC3002ADC.5, OK3B.COL, SPI_OUT.1
- net EXT_MOTOR_A: now also IC3.VI; no longer VREG.IN
- net EXT_MOTOR_GND: now also C1.2, CHANNEL_1_ADC.2, CHANNEL_3_ADC.2, CHANNEL_4_ADC.2, IC3.GND, IC3.GND@1, OK4A.EMIT, OK4B.EMIT, OK5A.EMIT, OK5B.EMIT, OK6A.C, U$2.AGND, U$2.DGND; no longer MPC3002ADC.4, MPC3002ADC.8, OK1C.EMIT, OK1D.EMIT, OK2C.EMIT, OK2D.EMIT, OK3C.C, VREG.GND
- net GND: now also C2.1, OK6A.EMIT, OK6B.EMIT, R1.2, R3.2, R33.2, R34.1, R35.1, R36.1, R37.1, R38.1, SENSOR_GND.1, SENSOR_GND.2; no longer JP10.2, JP11.2, JP12.2, JP13.2, OK3C.EMIT, OK3D.EMIT, R1.1, R3.1, X1.2, X1.3
- net MISO: now also OK6A.COL; no longer OK3C.COL
- net MOSI: now also OK5B.A; no longer OK3B.A
- net MOT_CONTROL_A_1: now also Q2.G, R1.1; no longer OK1B.A
- net MOT_CONTROL_A_2: now also Q5.G, R6.2; no longer OK2B.A
- net MOT_CONTROL_B_1: now also Q4.G, R3.1; no longer OK1C.A
- net MOT_CONTROL_B_2: now also Q6.G, R7.2; no longer OK2C.A
- net MOT_CONTROL_EN_1: now also Q1.G, R33.1; no longer OK1A.A
- net MOT_CONTROL_EN_2: now also Q3.G, R5.2; no longer OK2A.A
- net N$10: now also OK3A.C, Q5.D; no longer OK2B.C, R6.2
- net N$11: now also Q5.S, R37.2; no longer OK2C.C, R7.2
- net N$12: now also OK4B.C; no longer OK2D.C
- net N$13: now also OK5A.C; no longer OK3A.C
- net N$14: now also OK5B.C; no longer OK3B.C
- net N$18: now also OK2A.C, Q4.D; no longer CHANNEL_1_ADC.2, MPC3002ADC.3
- net N$19: now also OK4B.COL; no longer OK2D.COL
- net N$2: now also Q1.S, R2.2; no longer JP12.1, JP13.1, X1.4
- net N$28: now also OK2B.COL; no longer OK2A.COL
- net N$29: now also OK2A.COL; no longer OK1C.COL
- net N$30: now also OK3A.COL; no longer OK2B.COL
- net N$33: now also OK3B.COL; no longer OK2C.COL
- net N$34: now also OK6A.A; no longer OK3C.A
- net N$35: now also OK6B.A; no longer OK3D.A
- net N$36: now also OK6B.C; no longer OK3D.C
- net N$38: now also Q6.S, R38.2; no longer JP10.1, JP11.1, X1.1
- net N$41: now also OK3B.C, Q6.D; no longer IC1.PR0(XT2)
- net N$5: now also Q2.S, R34.2; no longer OK1A.C, R2.2
- net N$6: now also Q2.D; no longer R1.2
- net N$7: now also Q4.S, R36.2; no longer OK1C.C, R3.2
- net N$8: now also OK4A.C; no longer OK1D.C
- net N$9: now also OK2B.C, Q3.D; no longer OK2A.C, R5.2
- net OPTIONAL_OPTO_IN: now also IC1.PR0(XT2), OK6B.COL; no longer OK3D.COL
- net SCK: now also OK5A.A; no longer OK3A.A
- net SS1: now also OK4B.A; no longer OK2D.A
- net SS2: now also OK4A.A; no longer OK1D.A
Other:
- moved on the sheet: CHANNEL_1_ADC, CHANNEL_2_ADC, EXTERNAL_POWER_IN, IC2, LED1, LED2, LED3, MOTOR_1_OUT, MOTOR_2_OUT, OK1A, OK1B, OK2A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
